File: bistable-switch.brd (EAGLE design)
At the start: 13.9 x 17.8 mm, 13 parts, among them U1 CD4013BM, U2 AO3400, U3 AO3400

Commit message: update pcb
Parts:
- renumbered 3V3 to VCC
Changed lines of the file:
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@@
 </autorouter>
 <elements>
-<element name="3V3" library="BeagleBone_Blue_R3" library_urn="urn:adsk.eagle:library:5828899" package="B1,27" package3d_urn="urn:adsk.eagle:package:5829429/1" value="TPB1,27" x="1.143" y="1.143" smashed="yes">
+<element name="VCC" library="BeagleBone_Blue_R3" library_urn="urn:adsk.eagle:library:5828899" package="B1,27" package3d_urn="urn:adsk.eagle:package:5829429/1" value="TPB1,27" x="1.143" y="1.143" smashed="yes">
 <attribute name="NAME" x="1.778" y="2.032" size="0.6096" layer="25" ratio="10"/>
 <attribute name="TP_SIGNAL_NAME" value="" x="0.508" y="-0.762" size="1" layer="37"/>
@@
 <contactref element="S1" pad="4"/>
 <contactref element="C1" pad="2"/>
-<contactref element="3V3" pad="TP"/>
+<contactref element="VCC" pad="TP"/>
 <contactref element="U1" pad="14"/>
 <contactref element="D1" pad="1"/>
