File: bistable-switch.sch (EAGLE design)
At the start: 13 parts, among them U1 CD4013BM, U2 AO3400, U3 AO3400

Commit message: update pcb
Parts:
- renumbered 3V3 to VCC
Changed lines of the file:
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@@
 <part name="R1" library="Tubescreamer" library_urn="urn:adsk.eagle:library:41628504" deviceset="R-US_" device="R0805" package3d_urn="urn:adsk.eagle:package:42437559/3" value="10kOhm"/>
 <part name="C1" library="Tubescreamer" library_urn="urn:adsk.eagle:library:41628504" deviceset="C-US" device="C0805" package3d_urn="urn:adsk.eagle:package:42437565/3" value="100nF"/>
-<part name="3V3" library="BeagleBone_Blue_R3" library_urn="urn:adsk.eagle:library:5828899" deviceset="TP" device="B1,27" package3d_urn="urn:adsk.eagle:package:5829429/1"/>
+<part name="VCC" library="BeagleBone_Blue_R3" library_urn="urn:adsk.eagle:library:5828899" deviceset="TP" device="B1,27" package3d_urn="urn:adsk.eagle:package:5829429/1"/>
 <part name="GND" library="BeagleBone_Blue_R3" library_urn="urn:adsk.eagle:library:5828899" deviceset="TP" device="B1,27" package3d_urn="urn:adsk.eagle:package:5829429/1"/>
 <part name="DR" library="BeagleBone_Blue_R3" library_urn="urn:adsk.eagle:library:5828899" deviceset="TP" device="B1,27" package3d_urn="urn:adsk.eagle:package:5829429/1"/>
@@
 <attribute name="VALUE" x="37.211" y="92.456" size="1.778" layer="96" rot="R90"/>
 </instance>
-<instance part="3V3" gate="G$1" x="63.5" y="68.58" smashed="yes">
+<instance part="VCC" gate="G$1" x="63.5" y="68.58" smashed="yes">
 <attribute name="NAME" x="62.23" y="69.85" size="1.778" layer="95"/>
 </instance>
@@
 <wire x1="38.1" y1="91.44" x2="43.18" y2="91.44" width="0.1524" layer="91"/>
 <wire x1="43.18" y1="91.44" x2="43.18" y2="78.74" width="0.1524" layer="91"/>
-<pinref part="3V3" gate="G$1" pin="TP"/>
+<pinref part="VCC" gate="G$1" pin="TP"/>
 <pinref part="U1" gate="A" pin="VDD"/>
 <wire x1="43.18" y1="66.04" x2="63.5" y2="66.04" width="0.1524" layer="91"/>
